File: PCB/StenoWing.kicad_pcb (KiCad board)
At the start: 2 copper layers, 235.4 x 78.8 mm, 94 parts, among them SW1 Blank, SW11 Blank, SW12 Blank, SW13 Blank, SW14 Blank, SW15 Blank, SW16 Blank, SW17 Blank, SW18 Blank, SW19 Blank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

Commit message: StenoWing V2
Parts:
- removed the REF** at (138.8, 121.3)
- mcu: footprint footprints:Frood_PinHeader_2x13+5_P2.54mm_Labels_Top -> Symbol:Frood_PinHeader_2x13+5_P2.54mm_Labels_Top_LESS_PINS
Routing:
- net GND: track 89.8 -> 633.2 mm, vias 72 -> 81
- net SW_D15: track 35.7 -> 40.9 mm
- net Col_4: track 133.7 -> 136.7 mm
- net col_7: track 161.3 -> 159.6 mm
- net led24-out: track 39.8 -> 40.5 mm
Other:
- board text added: "Model: StenoWing28 (MX/Choc V2) Designed by: github.com/gzowski"
- board text added: "StenoWing v2"
- board text removed: "Model: StenoWing28 (MX/Choc V1) Designed by: github.com/gzowski"
- board text removed: "StenoWing"

Commit message: Changes
Routing:
- net vsys: track 694.8 -> 691.8 mm
Changed lines of the file:
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@@
-	)
-	(segment
-		(start 138.7 104.15)
-		(end 138.7 119.95)
-		(width 0.5)
-		(layer "B.Cu")
-		(net 25)
 	)
 	(segment
@@
 	)
 	(segment
+		(start 138.7 104.15)
+		(end 138.7 121.09)
+		(width 0.5)
+		(layer "B.Cu")
+		(net 25)
+	)
+	(segment
 		(start 46.823115 112.263115)
 		(end 46.823115 110.850261)
@@
 		(layer "B.Cu")
 		(net 25)
-	)
-	(segment
-		(start 138.7 119.95)
-		(end 138.7 124.03193)
-		(width 0.3)
-		(layer "B.Cu")
-		(net 25)
